Commit message: asdjfkasdf

File: robotplus_moveit_config/config/gazebo_robot.urdf (robot description, URDF)
Before this commit: robot robot, 15 links, 14 joints
Joints:
- joint base_link_fixed: origin xyz=0 0.05 0.77 rpy=0 0 -1.4509 -> xyz=0 0 0.77 rpy=0 0 -1.4509
- joint marker_fixed: origin xyz=1.36 2.42 0.06 rpy=0 0 0 -> xyz=1.14 2.05 -0.14 rpy=0 -0.3490658503988659 0

Commit message: 250509

File: robotplus_moveit_config/config/gazebo_robot.urdf (robot description, URDF)
Before this commit: robot robot, 15 links, 14 joints
Joints:
- joint base_link_fixed: origin xyz=0 0 0.77 rpy=0 0 -1.5709 -> xyz=0.1 -0.2 0.77 rpy=0 0 -1.4509
