Commit message: 250507

File: robotplus_moveit_config/config/gazebo_robot2.urdf (robot description, URDF)
Before this commit: robot robot, 15 links, 14 joints
Links:
- removed link base
- removed link base_link
- removed link cam
- removed link cam_optical
- removed link end
- removed link gripper_cam_jig
- removed link link1
- removed link link2
- removed link link3
- removed link link4
- removed link link5
- removed link link6
- removed link machine
- removed link marker_plate
- added link base2, mass 0.1; collision mesh filename=package://robotplus_description/meshes/base.STL; visual mesh filename=package://robotplus_description/meshes/base.STL
- added link base_link2, mass 0.1; collision mesh filename=package://robotplus_description/meshes/UR10e/base_link.STL; visual mesh filename=package://robotplus_description/meshes/UR10e/base_link.STL
- added link cam2, mass 0.1; collision mesh filename=package://robotplus_description/meshes/cam.STL; visual mesh filename=package://robotplus_description/meshes/cam.STL
- added link end2
- added link gripper_cam_jig2, mass 0.1; collision mesh filename=package://robotplus_description/meshes/gripper_cam_jig.STL; visual mesh filename=package://robotplus_description/meshes/gripper_cam_jig.STL
- added link link21, mass 0.1; collision mesh filename=package://robotplus_description/meshes/UR10e/link1.STL; visual mesh filename=package://robotplus_description/meshes/UR10e/link1.STL
- added link link22, mass 0.1; collision mesh filename=package://robotplus_description/meshes/UR10e/link2.STL; visual mesh filename=package://robotplus_description/meshes/UR10e/link2.STL
- added link link23, mass 0.1; collision mesh filename=package://robotplus_description/meshes/UR10e/link3.STL; visual mesh filename=package://robotplus_description/meshes/UR10e/link3.STL
- added link link24, mass 0.1; collision mesh filename=package://robotplus_description/meshes/UR10e/link4.STL; visual mesh filename=package://robotplus_description/meshes/UR10e/link4.STL
- added link link25, mass 0.1; collision mesh filename=package://robotplus_description/meshes/UR10e/link5.STL; visual mesh filename=package://robotplus_description/meshes/UR10e/link5.STL
- added link link26, mass 0.1; collision mesh filename=package://robotplus_description/meshes/UR10e/link6.STL; visual mesh filename=package://robotplus_description/meshes/UR10e/link6.STL
Joints:
- removed joint base_fixed
- removed joint base_link_fixed
- removed joint cam_joint
- removed joint jig_cam
- removed joint link6_end
- removed joint link6_jig
- removed joint machine_fixed
- removed joint marker_fixed
- removed joint q1
- removed joint q2
- removed joint q3
- removed joint q4
- removed joint q5
- removed joint q6
- added joint base_fixed2: type fixed, parent base_link2, child base2, origin xyz=0.42 0.62 0 rpy=-1.5709 0 3.1416
- added joint base_link_fixed2: type fixed, parent world, child base_link2, origin xyz=0 0 0.77 rpy=0 0 -1.4509
- added joint jig_cam2: type fixed, parent gripper_cam_jig2, child cam2, origin xyz=-0.0583225279657438 0 -0.0820000000000001 rpy=3.14159265358979 0 1.5707963267949, axis 0 0 0
- added joint link26_end2: type fixed, parent link26, child end2, origin xyz=0 0 0.12 rpy=3.1415 0 1.5708, axis 0 0 0
- added joint link26_jig2: type fixed, parent link26, child gripper_cam_jig2, origin xyz=0 0 0.12 rpy=3.1416 0 1.5709, axis 0 0 0
- added joint q21: type revolute, parent base_link2, child link21, origin xyz=0 0 0 rpy=0 0 0, axis 0 0 1, limit lower=-3.14 upper=3.14 effort=100 velocity=10
- added joint q22: type revolute, parent link21, child link22, origin xyz=0 0 0.1807 rpy=1.5708 1.5708 0, axis 0 0 1, limit lower=-3.14 upper=3.14 effort=100 velocity=10
- added joint q23: type revolute, parent link22, child link23, origin xyz=-0.6127 0 0 rpy=0 0 0, axis 0 0 1, limit lower=-3.14 upper=3.14 effort=100 velocity=10
- added joint q24: type revolute, parent link23, child link24, origin xyz=-0.57155 0 0 rpy=0 0 -1.5708, axis 0 0 1, limit lower=-3.14 upper=3.14 effort=100 velocity=10
- added joint q25: type revolute, parent link24, child link25, origin xyz=0 0 0.17415 rpy=1.5708 0 0, axis 0 0 1, limit lower=-3.14 upper=3.14 effort=100 velocity=10
- added joint q26: type revolute, parent link25, child link26, origin xyz=0 0 0.11985 rpy=-1.5708 0 0, axis 0 0 1, limit lower=-3.14 upper=3.14 effort=100 velocity=10

Commit message: position, rotation error correction

File: robotplus_moveit_config/config/gazebo_robot2.urdf (robot description, URDF)
Before this commit: robot robot, 12 links, 11 joints
Joints:
- joint base_link_fixed2: origin xyz=0 0 0.77 rpy=0 0 -1.4509 -> xyz=0.1 -0.2 0.77 rpy=0 0 -1.4509
